Commit message: Added camera collision

File: ws/src/robot_description/urdf/include/base_macro.urdf.xacro (robot description, xacro)
@@ -25,4 +25,10 @@
                 </material>
             </visual>
+            <collision>
+                <origin xyz="0 0 0" rpy="0 0 0"/>
+                <geometry>
+                    <mesh filename="package://robot_description/meshes/Oak-D/${model}.stl" />
+                </geometry>
+            </collision>
         </link>
         <joint name="${camera_name}_model_origin_joint" type="fixed">
