Commit message: Updated URDF

File: ws/src/robot_description/urdf/dashgo.urdf.xacro (robot description, xacro)
@@ -293,5 +293,5 @@
   <xacro:load_gripperSF attach_to="$(arg prefix)link_eef" xyz="0 0 0.007" rpy="-1.57 0 2.3554" />
   <xacro:include filename="$(find robot_description)/urdf/camera.urdf.xacro" />
-  <xacro:load_camera name="Cam1" attach_to="Base_Gripper" x="0.07" y="-0.05" z="0.0" r_p="-0.785398" r_r="1.5707" r_y="0.0" />
+  <xacro:load_camera name="Cam1" attach_to="Base_Gripper" x="0.0679" y="-0.03439" z="0.0" r_p="-0.785398" r_r="1.5707" r_y="0.0" />
   <xacro:load_camera name="Cam2" attach_to="Base" x="-0.085" y="-0.24" z="0.48" r_r="0.538132" r_p="0" r_y="-1.5708" />
 </robot>

File: ws/src/robot_description/urdf/gripper/gripperSF.urdf.xacro (robot description, xacro)
@@ -17,5 +17,5 @@
         <parent link="Base_Gripper" />
         <child link="end_effector_link" />
-        <origin xyz="0.0 -0.125 0" rpy="1.57 0 -1.57" />
+        <origin xyz="0.0 -0.05 0" rpy="1.57 0 -1.57" />
     </joint>
     <link

Commit message: Updated URDF and SRDF to fit navigation transforms

File: ws/src/robot_description/urdf/dashgo.urdf.xacro (robot description, xacro)
@@ -1,14 +1,14 @@
 <?xml version='1.0' encoding='utf-8'?>
 <robot xmlns:xacro="http://ros.org/wiki/xacro" name="dashgo">
-  <virtual_joint child_link="base_footprint" name="world_joint" parent_frame="odom" type="planar" />
-  <link name="base_footprint" />
+  <virtual_joint child_link="base_link" name="world_joint" parent_frame="base_footprint" type="planar" />
+  <!-- <link name="base_footprint" />
   <joint name="base_footprint_joint" type="fixed">
     <origin xyz="0 0 0" rpy="0 0 0" />
     <parent link="base_footprint" />
     <child link="base_link" />
-  </joint>
+  </joint> -->
   <link name="base_link" />
   <joint name="base_link_joint" type="fixed">
-    <origin xyz="0 0 0" rpy="0 0 0" />
+    <origin xyz="0 0 0" rpy="0 0 1.57" />
     <parent link="base_link" />
     <child link="Base" />

Commit message: URDF TMR2024 (includes fixes to base stl and camera position)

File: ws/src/robot_description/urdf/dashgo.urdf.xacro (robot description, xacro)
@@ -29,5 +29,5 @@
       <origin xyz="0 0 0" rpy="0 0 0" />
       <geometry>
-        <mesh filename="package://robot_description/meshes/Dashgo/dashgo_cubierta.stl" />
+        <mesh filename="package://robot_description/meshes/Dashgo/Base.STL" />
       </geometry>
       <material name="">
@@ -261,5 +261,5 @@
   </link>
   <joint name="Bra1Fix" type="fixed">
-    <origin xyz="0 0.054 0.4581" rpy="0 0 0" />
+    <origin xyz="0 0.044 0.4581" rpy="0 0 0" />
     <parent link="Base" />
     <child link="BaseBrazo" />
@@ -293,5 +293,5 @@
   <xacro:load_gripperSF attach_to="$(arg prefix)link_eef" xyz="0 0 0.007" rpy="-1.57 0 2.3554" />
   <xacro:include filename="$(find robot_description)/urdf/camera.urdf.xacro" />
-  <xacro:load_camera name="Cam1" attach_to="Base_Gripper" x="0.0679" y="-0.03439" z="0.0" r_p="-0.785398" r_r="1.5707" r_y="0.0" />
+  <xacro:load_camera name="Cam1" attach_to="Base_Gripper" x="0.068098" y="-0.035446" z="0.0" r_p="-0.785398" r_r="1.5707" r_y="0.0" />
   <xacro:load_camera name="Cam2" attach_to="Base" x="-0.085" y="-0.24" z="0.48" r_r="0.538132" r_p="0" r_y="-1.5708" />
 </robot>

Commit message: Full URDF update, corrections to ALL orientations and to Base STL.

File: ws/src/robot_description/urdf/dashgo.urdf.xacro (robot description, xacro)
@@ -10,14 +10,14 @@
   <link name="base_link" />
   <joint name="base_link_joint" type="fixed">
-    <origin xyz="0 0 0" rpy="0 0 1.57" />
+    <origin xyz="0 0 0" rpy="0 0 0" />
     <parent link="base_link" />
     <child link="Base" />
   </joint>
-  <link name="apriltag" />
+  <!-- <link name="apriltag" />
   <joint name="apriltag_joint" type="fixed">
     <origin xyz="0.06 0 0.06" rpy="3.14 -1.57 0" />
     <parent link="BaseBrazo" />
     <child link="apriltag" />
-  </joint>
+  </joint> -->
   <link name="Base">
     <inertial>
@@ -65,8 +65,8 @@
   </link>
   <joint name="Llanta1Cont" type="continuous">
-    <origin xyz="0.146 0.1155 0.0375" rpy="1.5708 0 1.5708" />
+    <origin xyz="-0.075244 0.166 0.0375" rpy="1.5708 0 3.1416" />
     <parent link="Base" />
     <child link="Llanta1" />
-    <axis xyz="0 0 1" />
+    <axis xyz="0 0 -1" />
   </joint>
   <link name="Llanta2">
@@ -93,8 +93,8 @@
   </link>
   <joint name="Llanta2Cont" type="continuous">
-    <origin xyz="-0.146 0.1155 0.0375" rpy="1.5708 0.020949 1.5708" />
+    <origin xyz="-0.075244 -0.166 0.0375" rpy="1.5708 0 3.1416" />
     <parent link="Base" />
     <child link="Llanta2" />
-    <axis xyz="0 0 1" />
+    <axis xyz="0 0 -1" />
   </joint>
   <link name="Loca1">
@@ -121,8 +121,8 @@
   </link>
   <joint name="Loca1Cont" type="continuous">
-    <origin xyz="-0.09 -0.072 0" rpy="1.5708 0 0" />
+    <origin xyz="0.11226 0.09 0.0025837" rpy="1.5708 0 -3.1152" />
     <parent link="Base" />
     <child link="Loca1" />
-    <axis xyz="0 1 0" />
+    <axis xyz="0 0 1" />
   </joint>
   <link name="LlantaLoca1">
@@ -149,8 +149,8 @@
   </link>
   <joint name="LlantaLoca1Cont" type="continuous">
-    <origin xyz="0 0.01 0" rpy="0 0 0" />
+    <origin xyz="0 0 0" rpy="0 0 0" />
     <parent link="Loca1" />
     <child link="LlantaLoca1" />
-    <axis xyz="1 0 0" />
+    <axis xyz="0 0 1" />
   </joint>
   <link name="Loca2">
@@ -177,8 +177,8 @@
   </link>
   <joint name="Loca2Cont" type="continuous">
-    <origin xyz="0.09 -0.072 0" rpy="1.5708 0 0.11924" />
+    <origin xyz="0.11226 -0.09 0.0025837" rpy="1.5708 0 -3.1152" />
     <parent link="Base" />
     <child link="Loca2" />
-    <axis xyz="0 1 0" />
+    <axis xyz="0 0 1" />
   </joint>
   <link name="LlantaLoca2">
@@ -205,8 +205,8 @@
   </link>
   <joint name="LlantaLoca2Cont" type="continuous">
-    <origin xyz="0 0.01 0" rpy="-0.88606 0 0" />
+    <origin xyz="0 0 0" rpy="0 0 0" />
     <parent link="Loca2" />
     <child link="LlantaLoca2" />
-    <axis xyz="1 0 0" />
+    <axis xyz="0 0 1" />
   </joint>
   <link name="Lidar">
@@ -233,5 +233,5 @@
   </link>
   <joint name="Lidar1Cont" type="continuous">
-    <origin xyz="0 -0.11 0.12" rpy="1.5708 0 0" />
+    <origin xyz="0.15026 0 0.1325" rpy="3.1416 0 0" />
     <parent link="Base" />
     <child link="Lidar" />
@@ -260,6 +260,6 @@
     </collision>
   </link>
-  <joint name="Bra1Fix" type="fixed">
-    <origin xyz="0 0.044 0.4581" rpy="0 0 0" />
+  <joint name="basebrazo_joint" type="fixed">
+    <origin xyz="-0.0055 0 0.458" rpy="0 0 1.57" />
     <parent link="Base" />
     <child link="BaseBrazo" />
@@ -294,4 +294,20 @@
   <xacro:include filename="$(find robot_description)/urdf/camera.urdf.xacro" />
   <xacro:load_camera name="Cam1" attach_to="Base_Gripper" x="0.068098" y="-0.035446" z="0.0" r_p="-0.785398" r_r="1.5707" r_y="0.0" />
-  <xacro:load_camera name="Cam2" attach_to="Base" x="-0.085" y="-0.24" z="0.48" r_r="0.538132" r_p="0" r_y="-1.5708" />
+  <!-- <xacro:load_camera name="Cam2" attach_to="Base" x="-0.085" y="-0.24" z="0.48" r_r="0.538132" r_p="0" r_y="-1.5708" /> -->
+  <!-- OakD Pro Camera -->
+  <xacro:arg name="add_oakd1" default="false" />
+  <xacro:arg name="oakd1_camera_name"   default="oakd-pro" />
+  <xacro:arg name="oakd1_camera_model"  default="OAK-D-PRO" />
+  <xacro:arg name="oakd1_base_frame"    default="oak-d_frame" />
+  <xacro:arg name="oakd1_parent_frame"  default="Base" />
+  <xacro:arg name="oakd1_cam_pos_x"     default="0.260989676" />
+  <xacro:arg name="oakd1_cam_pos_y"     default="0.000295007" />
+  <xacro:arg name="oakd1_cam_pos_z"     default="0.481840697" />
+  <xacro:arg name="oakd1_cam_roll"      default="0.0" />
+  <xacro:arg name="oakd1_cam_pitch"     default="0.0" />
+  <xacro:arg name="oakd1_cam_yaw"       default="0.0" />
+  <xacro:include filename="$(find depthai_descriptions)/urdf/include/depthai_macro.urdf.xacro"/>
+  <xacro:if value="$(arg add_oakd1)">
+    <xacro:depthai_camera camera_name="$(arg oakd1_camera_name)" parent="$(arg oakd1_parent_frame)" camera_model="$(arg oakd1_camera_model)" base_frame="$(arg oakd1_base_frame)" cam_pos_x="$(arg oakd1_cam_pos_x)" cam_pos_y="$(arg oakd1_cam_pos_y)" cam_pos_z="$(arg oakd1_cam_pos_z)" cam_roll="$(arg oakd1_cam_roll)" cam_pitch="$(arg oakd1_cam_pitch)" cam_yaw="$(arg oakd1_cam_yaw)" />
+  </xacro:if>
 </robot>

Commit message: multiple heavy additions had to be made in the urdf in order for it to barely work... even though, probably a separated urdf must be done for simulation purposes, with its own launchers

File: ws/src/robot_description/urdf/dashgo.urdf.xacro (robot description, xacro)
@@ -2,10 +2,10 @@
 <robot xmlns:xacro="http://ros.org/wiki/xacro" name="dashgo">
   <virtual_joint child_link="base_link" name="world_joint" parent_frame="base_footprint" type="planar" />
-  <!-- <link name="base_footprint" />
+  <link name="base_footprint" />
   <joint name="base_footprint_joint" type="fixed">
-    <origin xyz="0 0 0" rpy="0 0 0" />
+    <origin xyz="0 0 0.1" rpy="0 0 0" />
     <parent link="base_footprint" />
     <child link="base_link" />
-  </joint> -->
+  </joint>
   <link name="base_link" />
   <joint name="base_link_joint" type="fixed">
@@ -23,6 +23,6 @@
     <inertial>
       <origin xyz="-0.0421641375528847 0.0262460783517876 0.278949374295985" rpy="0 0 0" />
-      <mass value="26.7355250620724" />
-      <inertia ixx="0.418467609556011" ixy="0.0235787657447133" ixz="8.3665476036404E-06" iyy="0.302793463787765" iyz="0.000125414849304393" izz="0.482705153704045" />
+      <mass value="99.7355250620724" />
+      <inertia ixx="0.01" ixy="0.0" ixz="0.0" iyy="0.01" iyz="0.0" izz="0.01"/>
     </inertial>
     <visual>
@@ -46,5 +46,5 @@
       <origin xyz="4.02455846426619E-16 6.59194920871187E-16 0.0200000000000003" rpy="0 0 0" />
       <mass value="0.528918539158378" />
-      <inertia ixx="0.000631308353030454" ixy="-1.64320882748444E-36" ixz="1.72050413075699E-18" iyy="0.000631308353030454" iyz="-1.31827511759964E-36" izz="0.00112157176228534" />
+      <inertia ixx="0.01" ixy="0.0" ixz="0.0" iyy="0.01" iyz="0.0" izz="0.01"/>
     </inertial>
     <visual>
@@ -74,5 +74,5 @@
       <origin xyz="-1.38777878078145E-17 -1.11022302462516E-16 -0.02" rpy="0 0 0" />
       <mass value="0.528918539158378" />
-      <inertia ixx="0.000631308353030454" ixy="-8.470329472543E-22" ixz="-9.10263751530836E-20" iyy="0.000631308353030454" iyz="4.50857846912387E-20" izz="0.00112157176228534" />
+      <inertia ixx="0.01" ixy="0.0" ixz="0.0" iyy="0.01" iyz="0.0" izz="0.01"/>
     </inertial>
     <visual>
@@ -102,5 +102,5 @@
       <origin xyz="0 0.0345546529721542 -2.77555756156289E-17" rpy="0 0 0" />
       <mass value="0.0167352759899297" />
-      <inertia ixx="7.54150196205056E-06" ixy="1.29419148906084E-21" ixz="-8.52898332671465E-22" iyy="5.85653067123054E-06" iyz="-1.78257050125666E-21" izz="7.09027556219276E-06" />
+      <inertia ixx="0.01" ixy="0.0" ixz="0.0" iyy="0.01" iyz="0.0" izz="0.01"/>
     </inertial>
     <visual>
@@ -130,5 +130,5 @@
       <origin xyz="1.38777878078145E-17 -0.00741632050454701 1.38777878078145E-17" rpy="0 0 0" />
       <mass value="0.0694291976443344" />
-      <inertia ixx="3.17985725211052E-05" ixy="-5.21349495168481E-38" ixz="3.52930394689292E-22" iyy="1.95153903045283E-05" iyz="7.67877008722515E-41" izz="1.95153903045283E-05" />
+      <inertia ixx="0.01" ixy="0.0" ixz="0.0" iyy="0.01" iyz="0.0" izz="0.01"/>
     </inertial>
     <visual>
@@ -158,5 +158,5 @@
       <origin xyz="0 0.0345546529721542 2.77555756156289E-17" rpy="0 0 0" />
       <mass value="0.0167352759899297" />
-      <inertia ixx="7.54150196205057E-06" ixy="-2.82359729101002E-21" ixz="3.17637355220363E-22" iyy="5.85653067123054E-06" iyz="2.05773707188381E-21" izz="7.09027556219276E-06" />
+      <inertia ixx="0.01" ixy="0.0" ixz="0.0" iyy="0.01" iyz="0.0" izz="0.01"/>
     </inertial>
     <visual>
@@ -186,5 +186,5 @@
       <origin xyz="0 -0.00469061857919597 -0.00574455456677592" rpy="0 0 0" />
       <mass value="0.0694291976443344" />
-      <inertia ixx="3.17985725211052E-05" ixy="-8.15269211732264E-21" ixz="4.2351647362715E-22" iyy="1.95153903045283E-05" iyz="-1.6940658945086E-21" izz="1.95153903045284E-05" />
+      <inertia ixx="0.01" ixy="0.0" ixz="0.0" iyy="0.01" iyz="0.0" izz="0.01"/>
     </inertial>
     <visual>
@@ -214,5 +214,5 @@
       <origin xyz="-9.49517221724887E-50 0.0125 -1.38777878078145E-17" rpy="0 0 0" />
       <mass value="0.0962112750161874" />
-      <inertia ixx="3.44757068808005E-05" ixy="8.13422838622583E-38" ixz="1.3254524700622E-52" iyy="5.89294059474148E-05" iyz="-6.00991536754997E-37" izz="3.44757068808005E-05" />
+      <inertia ixx="0.01" ixy="0.0" ixz="0.0" iyy="0.01" iyz="0.0" izz="0.01"/>
     </inertial>
     <visual>
@@ -232,6 +232,6 @@
     </collision>
   </link>
-  <joint name="Lidar1Cont" type="continuous">
-    <origin xyz="0.15026 0 0.1325" rpy="3.1416 0 0" />
+  <joint name="Lidar1Cont" type="fixed">
+    <origin xyz="0.15026 0 0.1325" rpy="0 0 0" />
     <parent link="Base" />
     <child link="Lidar" />
@@ -242,5 +242,5 @@
       <origin xyz="-3.80430852558273E-17 -6.24500451351651E-17 -5.000000000005E-05" rpy="0 0 0" />
       <mass value="0.00121022002997899" />
-      <inertia ixx="1.17272637070328E-06" ixy="2.62532909257585E-23" ixz="-6.31088724176809E-28" iyy="1.17272637070328E-06" iyz="8.80890739742394E-43" izz="2.34545072437318E-06" />
+      <inertia ixx="0.01" ixy="0.0" ixz="0.0" iyy="0.01" iyz="0.0" izz="0.01"/>
     </inertial>
     <visual>
@@ -356,3 +356,100 @@
     <xacro:depthai_camera camera_name="$(arg oakd1_camera_name)" parent="$(arg oakd1_parent_frame)" camera_model="$(arg oakd1_camera_model)" base_frame="$(arg oakd1_base_frame)" cam_pos_x="$(arg oakd1_cam_pos_x)" cam_pos_y="$(arg oakd1_cam_pos_y)" cam_pos_z="$(arg oakd1_cam_pos_z)" cam_roll="$(arg oakd1_cam_roll)" cam_pitch="$(arg oakd1_cam_pitch)" cam_yaw="$(arg oakd1_cam_yaw)" />
   </xacro:if>
+  <gazebo>
+    <plugin name="object_controller" filename="libgazebo_ros_planar_move.so">
+      <commandTopic>cmd_vel</commandTopic>
+      <odometryTopic>odom</odometryTopic>
+      <odometryFrame>odom</odometryFrame>
+      <odometryRate>20.0</odometryRate>
+      <robotBaseFrame>base_footprint</robotBaseFrame>
+    </plugin>
+  </gazebo>
+   <!-- hokuyo -->
+   <gazebo reference="Lidar">
+    <sensor type="gpu_ray" name="head_hokuyo_sensor">
+      <pose>0 0 0 0 0 0</pose>
+      <visualize>true</visualize>
+      <update_rate>40</update_rate>
+      <ray>
+        <scan>
+          <horizontal>
+            <samples>720</samples>
+            <resolution>1</resolution>
+            <min_angle>-3.1416</min_angle>
+            <max_angle>3.1416</max_angle>
+          </horizontal>
+        </scan>
+        <range>
+          <min>0.4</min>
+          <max>30.0</max>
+          <resolution>0.01</resolution>
+        </range>
+        <noise>
+          <type>gaussian</type>
+          <!-- Noise parameters based on published spec for Hokuyo laser
+               achieving "+-30mm" accuracy at range < 10m.  A mean of 0.0m and
+               stddev of 0.01m will put 99.7% of samples within 0.03m of the true
+               reading. -->
+          <mean>0.0</mean>
+          <stddev>0.01</stddev>
+        </noise>
+      </ray>
+      <plugin name="gazebo_ros_head_hokuyo_controller" filename="libgazebo_ros_gpu_laser.so">
+        <topicName>scan</topicName>
+        <frameName>Base</frameName>
+      </plugin>
+    </sensor>
+  </gazebo>
+  <gazebo reference="base_footprint">
+    <selfCollide>false</selfCollide>
+    <gravity>0</gravity>
+  </gazebo>
+  <gazebo reference="base_link">
+    <selfCollide>false</selfCollide>
+    <gravity>0</gravity>
+  </gazebo>
+  <gazebo reference="Base">
+    <selfCollide>false</selfCollide>
+    <gravity>0</gravity>
+  </gazebo>
+  <gazebo reference="Llanta1">
+    <selfCollide>false</selfCollide>
+    <gravity>0</gravity>
+  </gazebo>
+  <gazebo reference="Llanta2">
+    <selfCollide>false</selfCollide>
+    <gravity>0</gravity>
+  </gazebo>
+  <gazebo reference="Loca1">
+    <selfCollide>false</selfCollide>
+    <gravity>0</gravity>
+  </gazebo>
+  <gazebo reference="LlantaLoca1">
+    <selfCollide>false</selfCollide>
+    <gravity>0</gravity>
+  </gazebo>
+  <gazebo reference="Loca2">
+    <selfCollide>false</selfCollide>
+    <gravity>0</gravity>
+  </gazebo>
+  <gazebo reference="LlantaLoca2">
+    <selfCollide>false</selfCollide>
+    <gravity>0</gravity>
+  </gazebo>
+  <gazebo reference="Lidar">
+    <selfCollide>false</selfCollide>
+    <gravity>0</gravity>
+  </gazebo>
+  <gazebo reference="BaseBrazo">
+    <selfCollide>false</selfCollide>
+    <gravity>0</gravity>
+  </gazebo>
+  <gazebo reference="Cam1">
+    <selfCollide>false</selfCollide>
+    <gravity>0</gravity>
+  </gazebo>
+  <gazebo reference="Lidar">
+    <selfCollide>false</selfCollide>
+    <gravity>0</gravity>
+  </gazebo>
 </robot>

File: ws/src/robot_description/urdf/gripper/gripper.urdf.xacro (robot description, xacro)
@@ -287,3 +287,43 @@
     </joint>
   </xacro:macro>
+  <gazebo reference="Base_Gripper">
+    <selfCollide>false</selfCollide>
+    <gravity>0</gravity>
+  </gazebo>
+  <gazebo reference="end_effector_link">
+    <selfCollide>false</selfCollide>
+    <gravity>0</gravity>
+  </gazebo>
+  <gazebo reference="Servo1">
+    <selfCollide>false</selfCollide>
+    <gravity>0</gravity>
+  </gazebo>
+  <gazebo reference="Dedo1">
+    <selfCollide>false</selfCollide>
+    <gravity>0</gravity>
+  </gazebo>
+  <gazebo reference="Servo2">
+    <selfCollide>false</selfCollide>
+    <gravity>0</gravity>
+  </gazebo>
+  <gazebo reference="Dedo2">
+    <selfCollide>false</selfCollide>
+    <gravity>0</gravity>
+  </gazebo>
+  <gazebo reference="Rev1Servo">
+    <selfCollide>false</selfCollide>
+    <gravity>0</gravity>
+  </gazebo>
+  <gazebo reference="Rev2Servo">
+    <selfCollide>false</selfCollide>
+    <gravity>0</gravity>
+  </gazebo>
+  <gazebo reference="Fix1Dedo">
+    <selfCollide>false</selfCollide>
+    <gravity>0</gravity>
+  </gazebo>
+  <gazebo reference="Fix2Dedo">
+    <selfCollide>false</selfCollide>
+    <gravity>0</gravity>
+  </gazebo>
 </robot>
